File: BB.kicad_sch (KiCad schematic)
At the start: 61 parts, among them J10 Conn_01x01, J11 Conn_01x01, J12 Conn_01x01, J9 Conn_01x01, Q1 HYG080N10LS1C2, Q2 HYG080N10LS1C2, Q3 HYG080N10LS1C2, Q4 HYG080N10LS1C2, U1 UCC27211ADRMR, U18 UCC27519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

Commit message: 更改所有封装为SOD-323的1N4148W为1N4148WS 添加分压器的钳位二极管
Parts:
- D1, D2, D3, D4, D5, D6, D7, D8: value 1N4148W -> 1N4148WS
Changed lines of the file:
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@@
 			)
 		)
-		(property "Value" "1N4148W"
+		(property "Value" "1N4148WS"
 			(at 268.986 127 0)
 			(effects
@@
 			)
 		)
-		(property "Value" "1N4148W"
+		(property "Value" "1N4148WS"
 			(at 185.42 124.46 0)
 			(effects
@@
 			)
 		)
-		(property "Value" "1N4148W"
+		(property "Value" "1N4148WS"
 			(at 185.42 116.84 0)
 			(effects
@@
 			)
 		)
-		(property "Value" "1N4148W"
+		(property "Value" "1N4148WS"
 			(at 256.032 127 0)
 			(effects
@@
 			)
 		)
-		(property "Value" "1N4148W"
+		(property "Value" "1N4148WS"
 			(at 240.792 104.14 0)
 			(effects
@@
 			)
 		)
-		(property "Value" "1N4148W"
+		(property "Value" "1N4148WS"
 			(at 253.746 104.14 0)
 			(effects
@@
 			)
 		)
-		(property "Value" "1N4148W"
+		(property "Value" "1N4148WS"
 			(at 93.98 124.46 0)
 			(effects
@@
 			)
 		)
-		(property "Value" "1N4148W"
+		(property "Value" "1N4148WS"
 			(at 93.98 116.84 0)
 			(effects
