File: SENSE.kicad_sch (KiCad schematic)
At the start: 12 parts, among them U16 INA241A3xDDF, U17 INA241A3xDDF, U20 SGM8551XN, U21 SGM8551XN

Commit message: 更改所有封装为SOD-323的1N4148W为1N4148WS 添加分压器的钳位二极管
Parts:
- added D16, D17, D18, D19: 1N4148WS, Diode_SMD:D_SOD-323, symbol Diode:1N4148WS
Connections:
- net GNDA: now also D17.2 (A), D19.2 (A)
- net InputVsense+: now also D16.2 (A), D17.1 (K)
- net OutputVsense+: now also D18.2 (A), D19.1 (K)
- net VANA: now also D16.1 (K), D18.1 (K)
