File: MCU_MISC2.kicad_sch (KiCad schematic)
At the start: 19 parts, among them J1 USB_B, J2 USB_C_Receptacle_USB2.0_16P, J3 Conn_02x16_Odd_Even, Q5 S8050, U5 TPD4E05U06DQA

Commit message: 添加蜂鸣器IO及走线，更改PINMUX配图
Parts:
- added BZ1: Buzzer_DummyPIn3, 1MyFootPrint:Buzzer_5020_MetalHole, symbol 1MySymblesFromLCSC:Buzzer_DummyPIn3
- added C92: 1uF, Capacitor_SMD:C_0603_1608Metric, symbol Device:C
- added Q7: S8050, Package_TO_SOT_SMD:SOT-23, symbol 1MyRandom:S8050
- added R70: 0R, Resistor_SMD:R_0603_1608Metric, symbol Device:R
- added R71: 4.7k, Resistor_SMD:R_0603_1608Metric, symbol Device:R
- added R72: 100, Resistor_SMD:R_0603_1608Metric, symbol Device:R
Connections:
- net +3.3V: now also C92.1, R70.1
- net GND: now also BZ1.3 (DUM), C92.2, Q7.2 (E), R71.1
- new net: Q7.1 (B), R71.2, R72.1
- new net: BZ1.1 (+), R70.2
- new net: BZ1.2 (-), Q7.3 (C)
- new net BEEP: R72.2
Other:
- note added: "蜂鸣器"
