File: HardwareProject/MCU_IO_D.kicad_sch (KiCad schematic)
At the start: 2 parts, among them U4 HPM6P41IPB1

Commit message: rev4修改核心供电前保存（当前SYR838）
Parts:
- C105: renamed from C18; value 100nF,10V -> 100nF,50V
- renumbered U4 to U16
Changed lines of the file:
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@@
 		(dnp no)
 		(fields_autoplaced yes)
-		(property "Reference" "U4"
+		(property "Reference" "U16"
 			(at 265.43 95.8849 0)
 			(effects
@@
 			(project "HPM6P41_BB"
 				(path "/714b8a30-f9a7-49d4-a000-bc20c4884c7a/4759a0c1-ad86-4fab-9152-87dbcf52a213"
-					(reference "U4")
+					(reference "U16")
 					(unit 5)
 				)
@@
 		(dnp no)
 		(fields_autoplaced yes)
-		(property "Reference" "#PWR035"
+		(property "Reference" "#PWR0196"
 			(at 33.02 45.72 0)
 			(effects
@@
 			(project "HPM6P41_BB"
 				(path "/714b8a30-f9a7-49d4-a000-bc20c4884c7a/4759a0c1-ad86-4fab-9152-87dbcf52a213"
-					(reference "#PWR035")
+					(reference "#PWR0196")
 					(unit 1)
 				)
@@
 		(dnp no)
 		(fields_autoplaced yes)
-		(property "Reference" "#PWR036"
+		(property "Reference" "#PWR0197"
 			(at 33.02 55.88 0)
 			(effects
@@
 			(project "HPM6P41_BB"
 				(path "/714b8a30-f9a7-49d4-a000-bc20c4884c7a/4759a0c1-ad86-4fab-9152-87dbcf52a213"
-					(reference "#PWR036")
+					(reference "#PWR0197")
 					(unit 1)
 				)
@@
 		(on_board yes)
 		(dnp no)
-		(property "Reference" "C18"
+		(property "Reference" "C105"
 			(at 36.83 44.4499 0)
 			(effects
@@
 			)
 		)
-		(property "Value" "100nF,10V"
+		(property "Value" "100nF,50V"
 			(at 36.83 46.9899 0)
 			(effects
@@
 			(project "HPM6P41_BB"
 				(path "/714b8a30-f9a7-49d4-a000-bc20c4884c7a/4759a0c1-ad86-4fab-9152-87dbcf52a213"
-					(reference "C18")
+					(reference "C105")
 					(unit 1)
 				)
