File: HardwareProject/HPM6P41_BB.kicad_pcb (KiCad board)
At the start: 4 copper layers, 100 x 80.3 mm, 309 parts, among them J1 Conn_01x01, J10 排针, J11 Conn_ARM_JTAG_SWD_20, J12 排针, J13 排针, J2 Conn_01x01, J3 Conn_01x01, J4 Conn_01x01, J5 SMA, J6 SMA, J7 Conn_01x03, J8 Conn_01x03, J9 USB_C_Receptacle_USB2.0_16P, Q1 HYG080N10LS1C2, Q2 HYG080N10LS1C2, Q3 HYG080N10LS1C2, Q4 HYG080N10LS1C2, Q5 AO3400A, Q6 AO3400A, SW1 焊盘, SW2 Push_Button, SW3 Push_Button, SW4 Push_Button, U1 UCC27211ADRMR, U10 TPS54302, U11 INA241A3xDDF, U12 SGM8551XN, U13 SGM8551XN, U14 AT24C08C-SSHM-T, U15 TMP112xxDRL, U16 HPM6P41IPB1, U19 CA-IS3762HN, U2 UCC27211ADRMR, U20 TME-0505S, U21 SIT3088ETK, U22 TJA1044GTK/3Z, U23 TPD4E05U06DQA, U24 XC6206PxxxMR, U25 CA-IS3762HN, U26 TPD4E05U06DQA, U27 INA241A3xDDF, U3 UCC27517, U4 UCC27517, U5 SYR838, U6 SY8089, U7 LP5907MFX-3.3, U8 REF3030, U9 LM5164DDA, Y1 24MHz ±10ppm 6pF

Commit message: 小改丝印
Parts:
- added REF**: 7x1mm_导流条, 1MyFootPrint:7x1mm_导流条, B.Cu at (87.2, 53.0)
- added REF**: 7x1mm_导流条, 1MyFootPrint:7x1mm_导流条, B.Cu at (101.2, 44.4)
- added REF**: 7x1mm_导流条, 1MyFootPrint:7x1mm_导流条, B.Cu at (148.6, 42.0)
- added REF**: 7x1mm_导流条, 1MyFootPrint:7x1mm_导流条, B.Cu at (143.2, 39.6)
- added REF**: 7x1mm_导流条, 1MyFootPrint:7x1mm_导流条, B.Cu at (148.6, 47.0)
- added REF**: 7x1mm_导流条, 1MyFootPrint:7x1mm_导流条, B.Cu at (96.4, 39.8)
- added REF**: 7x1mm_导流条, 1MyFootPrint:7x1mm_导流条, B.Cu at (151.4, 44.4)
- added REF**: 7x1mm_导流条, 1MyFootPrint:7x1mm_导流条, B.Cu at (138.6, 46.9)
- added REF**: 7x1mm_导流条, 1MyFootPrint:7x1mm_导流条, B.Cu at (106.4, 44.5)
- added REF**: 7x1mm_导流条, 1MyFootPrint:7x1mm_导流条, B.Cu at (143.2, 50.0)
- added REF**: 7x1mm_导流条, 1MyFootPrint:7x1mm_导流条, B.Cu at (93.0, 50.0)
- added REF**: 7x1mm_导流条, 1MyFootPrint:7x1mm_导流条, B.Cu at (137.9, 40.8)
- added REF**: 7x1mm_导流条, 1MyFootPrint:7x1mm_导流条, B.Cu at (98.5, 47.0)
- added REF**: 7x1mm_导流条, 1MyFootPrint:7x1mm_导流条, B.Cu at (108.7, 44.5)
- added REF**: 7x1mm_导流条, 1MyFootPrint:7x1mm_导流条, B.Cu at (143.2, 44.4)
- added REF**: 7x1mm_导流条, 1MyFootPrint:7x1mm_导流条, B.Cu at (88.3, 39.8)
- added REF**: 7x1mm_导流条, 1MyFootPrint:7x1mm_导流条, B.Cu at (93.0, 44.4)
- added REF**: 7x1mm_导流条, 1MyFootPrint:7x1mm_导流条, B.Cu at (138.7, 51.8)
- added REF**: 7x1mm_导流条, 1MyFootPrint:7x1mm_导流条, B.Cu at (151.4, 39.6)
- added REF**: 7x1mm_导流条, 1MyFootPrint:7x1mm_导流条, B.Cu at (80.2, 39.8)
- added REF**: 7x1mm_导流条, 1MyFootPrint:7x1mm_导流条, B.Cu at (104.5, 39.8)
- added REF**: 7x1mm_导流条, 1MyFootPrint:7x1mm_导流条, B.Cu at (79.1, 53.0)
- added REF**: 7x1mm_导流条, 1MyFootPrint:7x1mm_导流条, B.Cu at (101.2, 50.0)
- added REF**: 7x1mm_导流条, 1MyFootPrint:7x1mm_导流条, B.Cu at (98.5, 42.0)
- added REF**: 7x1mm_导流条, 1MyFootPrint:7x1mm_导流条, B.Cu at (151.4, 50.0)
- renumbered BZ1 to BZ1-PY3, TP6 to GNDA, J5 to J5-PB1, J6 to J6-PB0, TP1 to PA12, TP2 to PA13, TP3 to PA14, TP4 to PA15
Routing:
- net Vdrv: track 105.0 -> 106.4 mm, vias 4 -> 5
- net VDD_SOC: vias 13 -> 14
- net GND: vias 73 -> 77
- net +3.3V: vias 22 -> 23
Other:
- board text added: "+3.3V"
- board text added: "+5V"
- board text added: "BT0"
- board text added: "BT1"
- board text added: "H1"
- board text added: "H2"
- board text added: "L1"
- board text added: "L2"
- board text added: "PY0~2"
- board text added: "VDD_SOC"
- board text added: "Vdrv"
- board text added: "Vin-PD6 Ipk-PD5/7 Iavg-PD8 Vout-PD9/10"

Commit message: Rev4保存
Routing:
- net VBUS: track 27.2 -> 24.7 mm
Changed lines of the file:
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@@
 	)
 	(gr_arc
-		(start 104.3 76)
-		(mid 103.960476 76.508134)
-		(end 103.361091 76.388909)
+		(start 104.8 76)
+		(mid 104.460476 76.508134)
+		(end 103.861091 76.388909)
 		(stroke
 			(width 0.15)
@@
 	)
 	(gr_line
-		(start 105.65 77.34792)
-		(end 104.15 77.34792)
+		(start 106 77.34792)
+		(end 104.5 77.34792)
 		(stroke
 			(width 0.15)
@@
 	)
 	(gr_arc
-		(start 105.65 77.34792)
-		(mid 106.25208 77.95)
-		(end 105.65 78.55208)
+		(start 106 77.34792)
+		(mid 106.60208 77.95)
+		(end 106 78.55208)
 		(stroke
 			(width 0.15)
@@
 	)
 	(gr_text "VDD_SOC"
-		(at 101.5 78.55 0)
+		(at 101.85 78.55 0)
 		(layer "F.SilkS")
 		(effects
@@
 	)
 	(gr_text "GND"
-		(at 102.15 77.35 0)
+		(at 102.5 77.35 0)
 		(layer "F.SilkS")
 		(effects
@@
 	)
 	(gr_text "GND"
-		(at 94.75 62.45 90)
+		(at 94.75 62.25 90)
 		(layer "F.SilkS")
 		(effects
@@
 	)
 	(gr_text "GND"
-		(at 104.25 74.05 270)
+		(at 104.75 74.05 270)
 		(layer "F.SilkS")
 		(effects
@@
 	)
 	(gr_text "+3.3V"
-		(at 101.8 73.95 300)
+		(at 102.3 73.95 300)
 		(layer "F.SilkS")
 		(effects
@@
 	)
 	(segment
-		(start 157.125 108.96)
-		(end 157.125 109.55)
-		(width 0.3048)
-		(layer "F.Cu")
-		(net 10)
-	)
-	(segment
 		(start 158.125 109.55)
 		(end 158.275 109.7)
@@
 	)
 	(segment
-		(start 156.775 109.55)
-		(end 157.125 109.55)
-		(width 0.3048)
-		(layer "F.Cu")
-		(net 10)
-	)
-	(segment
-		(start 157.125 109.55)
-		(end 158.125 109.55)
-		(width 0.3048)
+		(start 158.275 109.125)
+		(end 158.275 109.7)
+		(width 0.6096)
 		(layer "F.Cu")
 		(net 10)
@@
 	)
 	(segment
-		(start 156.625 108.960001)
-		(end 156.625 109.4)
-		(width 0.3048)
-		(layer "F.Cu")
-		(net 10)
-	)
-	(segment
 		(start 158.275 110.75)
 		(end 158.275 109.7)
@@
 	)
 	(segment
-		(start 156.625 109.4)
-		(end 156.775 109.55)
-		(width 0.3048)
+		(start 153.475 109.125)
+		(end 153.475 109.7)
+		(width 0.6096)
 		(layer "F.Cu")
 		(net 10)
@@
 	(segment
 		(start 153.475 109.7)
-		(end 153.475 109.125)
-		(width 0.6096)
-		(layer "B.Cu")
-		(net 10)
-	)
-	(segment
-		(start 153.475 109.7)
 		(end 154.675 109.7)
 		(width 0.6096)
@@
 		(width 0.6096)
 		(layer "B.Cu")
-		(net 10)
-	)
-	(segment
-		(start 158.275 109.125)
-		(end 158.275 109.7)
-		(width 0.6096)
-		(layer "B.Cu")
